File: schaltplan/schaltplan.kicad_sch (KiCad schematic)
At the start: 30 parts, among them J1 M1, J2 M2, J3 M4, J4 arduino pin 9, J5 arduino pin A8, J6 arduino pin A9, J7 arduino pin A7, J8 arduino pin 14, J9 M2, M1 Motor_DC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

Commit message: Add files via upload
Parts:
- R8: value 10k -> 100k
Changed lines of the file:
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@@
 			)
 		)
-		(property "Value" "10k"
+		(property "Value" "100k"
 			(at 80.01 104.1399 0)
 			(effects
